File: FT231x-Breakout.kicad_sch (KiCad schematic)
At the start: 26 parts, among them J1 USB JST, J2 CBUS, J3 SUPPLY, J4 TX/RX, J5 OTHER, Q1 BC558, Q2 BC558, SW1 SW_SPDT, U1 FT231XS

Commit message: Rev1.1
Signed-off-by: CTXz <ctx.xda@gmail.com>
Parts:
- D2: value LED -> RX LED
- D3: value LED -> TX LED
Other:
- note added: "Author: Patrick Pedersen <ctx.xda@gmail.com>"
- note added: "Broken-out/Exposed pins"
- note added: "FT231X USB-2-UART Breakout Board"
- note added: "JST XH 1x2"
- note added: "JST XH 1x3"
- note added: "LED mounted on enclosure"
- note added: "LED signal inverted since default UART state is HIGH"
- note added: "LEDs mounted on enclosure"
- note added: "Revision 1.1"
- note added: "Switch mounted on enclosure"
- company: (none) -> TU-DO Makerspace
- title: (none) -> FT231X USB 2 UART Breakout
- moved on the sheet: C1, C2, C3, C4, C5, C6, D1, D2, D3, J1, J2, J3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
