File: Kicad/FT231x-Breakout.kicad_pcb (KiCad board)
At the start: 2 copper layers, 70 x 100 mm, 30 parts, among them J1 USB JST, J2 CBUS, J3 SUPPLY, J4 TX/RX, J5 OTHER, Q1 BC558, Q2 BC558, SW1 SW_SPDT, U1 FT231XS

Commit message: Rev 1.2 + Added README
Signed-off-by: CTXz <ctx.xda@gmail.com>
Other:
- board text added: "Revision 1.2 Patrick Pedersen ctx.xda@gmail.com"
- board text removed: "Revision 1.1 Patrick Pedersen ctx.xda@gmail.com"
Changed lines of the file:
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@@
     (effects (font (size 1 1) (thickness 0.15)) (justify right bottom))
   )
-  (gr_text "Revision 1.1\nPatrick Pedersen\nctx.xda@gmail.com" (at 80.391 92.075) (layer "F.SilkS")
+  (gr_text "Revision 1.2\nPatrick Pedersen\nctx.xda@gmail.com" (at 80.391 92.075) (layer "F.SilkS")
     (effects (font (size 1 1) (thickness 0.15)) (justify left bottom))
   )
