File: Kicad/FT231x-Breakout.kicad_sch (KiCad schematic)
At the start: 26 parts, among them J1 USB JST, J2 CBUS, J3 SUPPLY, J4 TX/RX, J5 OTHER, Q1 BC558, Q2 BC558, SW1 SW_SPDT, U1 FT231XS

Commit message: Rev 1.2 + Added README
Signed-off-by: CTXz <ctx.xda@gmail.com>
Parts:
- R1: value 1k -> 10k
Other:
- note added: "Revision 1.2"
- note removed: "Revision 1.1"
Changed lines of the file:
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@@
     (effects (font (size 1 1)) (justify left bottom))
   )
-  (text "Revision 1.1" (at 18.415 33.02 0)
+  (text "Revision 1.2" (at 18.415 33.02 0)
     (effects (font (size 2 2)) (justify left bottom))
   )
@@
     (pin "2")
     (instances
-      (project "FTDIBreakout"
+      (project "FT231x-Breakout"
         (path "/3ba8e31e-6a12-4b2c-b7ff-be557fb7bb2f"
           (reference "D2") (unit 1)
@@
     (pin "1")
     (instances
-      (project "FTDIBreakout"
+      (project "FT231x-Breakout"
         (path "/3ba8e31e-6a12-4b2c-b7ff-be557fb7bb2f"
           (reference "#PWR02") (unit 1)
@@
     (pin "1")
     (instances
-      (project "FTDIBreakout"
+      (project "FT231x-Breakout"
         (path "/3ba8e31e-6a12-4b2c-b7ff-be557fb7bb2f"
           (reference "#PWR08") (unit 1)
@@
     (pin "1")
     (instances
-      (project "FTDIBreakout"
+      (project "FT231x-Breakout"
         (path "/3ba8e31e-6a12-4b2c-b7ff-be557fb7bb2f"
           (reference "#PWR022") (unit 1)
@@
     (pin "1")
     (instances
-      (project "FTDIBreakout"
+      (project "FT231x-Breakout"
         (path "/3ba8e31e-6a12-4b2c-b7ff-be557fb7bb2f"
           (reference "#PWR04") (unit 1)
@@
       (effects (font (size 1.27 1.27)) (justify left))
     )
-    (property "Value" "1k" (at 89.535 59.055 0)
+    (property "Value" "10k" (at 89.535 59.055 0)
       (effects (font (size 1.27 1.27)) (justify left))
     )
@@
     (pin "1")
     (instances
-      (project "FTDIBreakout"
+      (project "FT231x-Breakout"
         (path "/3ba8e31e-6a12-4b2c-b7ff-be557fb7bb2f"
           (reference "R1") (unit 1)
@@
     (pin "1")
     (instances
-      (project "FTDIBreakout"
+      (project "FT231x-Breakout"
         (path "/3ba8e31e-6a12-4b2c-b7ff-be557fb7bb2f"
           (reference "#PWR015") (unit 1)
@@
     (pin "1")
     (instances
-      (project "FTDIBreakout"
+      (project "FT231x-Breakout"
         (path "/3ba8e31e-6a12-4b2c-b7ff-be557fb7bb2f"
           (reference "#PWR020") (unit 1)
@@
     (pin "1")
     (instances
-      (project "FTDIBreakout"
+      (project "FT231x-Breakout"
         (path "/3ba8e31e-6a12-4b2c-b7ff-be557fb7bb2f"
           (reference "#PWR013") (unit 1)
@@
     (pin "2")
     (instances
-      (project "FTDIBreakout"
+      (project "FT231x-Breakout"
         (path "/3ba8e31e-6a12-4b2c-b7ff-be557fb7bb2f"
           (reference "D3") (unit 1)
@@
     (pin "2")
     (instances
-      (project "FTDIBreakout"
+      (project "FT231x-Breakout"
         (path "/3ba8e31e-6a12-4b2c-b7ff-be557fb7bb2f"
           (reference "J4") (unit 1)
@@
     (pin "8")
     (instances
-      (project "FTDIBreakout"
+      (project "FT231x-Breakout"
         (path "/3ba8e31e-6a12-4b2c-b7ff-be557fb7bb2f"
           (reference "U1") (unit 1)
@@
     (pin "1")
     (instances
-      (project "FTDIBreakout"
+      (project "FT231x-Breakout"
         (path "/3ba8e31e-6a12-4b2c-b7ff-be557fb7bb2f"
           (reference "R6") (unit 1)
@@
     (pin "1")
     (instances
-      (project "FTDIBreakout"
+      (project "FT231x-Breakout"
         (path "/3ba8e31e-6a12-4b2c-b7ff-be557fb7bb2f"
           (reference "#PWR014") (unit 1)
@@
     (pin "1")
     (instances
-      (project "FTDIBreakout"
+      (project "FT231x-Breakout"
         (path "/3ba8e31e-6a12-4b2c-b7ff-be557fb7bb2f"
           (reference "#PWR09") (unit 1)
@@
     (pin "2")
     (instances
-      (project "FTDIBreakout"
+      (project "FT231x-Breakout"
         (path "/3ba8e31e-6a12-4b2c-b7ff-be557fb7bb2f"
           (reference "C2") (unit 1)
@@
     (pin "1")
     (instances
-      (project "FTDIBreakout"
+      (project "FT231x-Breakout"
         (path "/3ba8e31e-6a12-4b2c-b7ff-be557fb7bb2f"
           (reference "R2") (unit 1)
@@
     (pin "1")
     (instances
-      (project "FTDIBreakout"
+      (project "FT231x-Breakout"
         (path "/3ba8e31e-6a12-4b2c-b7ff-be557fb7bb2f"
           (reference "C1") (unit 1)
@@
     (pin "1")
     (instances
-      (project "FTDIBreakout"
+      (project "FT231x-Breakout"
         (path "/3ba8e31e-6a12-4b2c-b7ff-be557fb7bb2f"
           (reference "#PWR018") (unit 1)
@@
     (pin "1")
     (instances
-      (project "FTDIBreakout"
+      (project "FT231x-Breakout"
         (path "/3ba8e31e-6a12-4b2c-b7ff-be557fb7bb2f"
           (reference "R7") (unit 1)
@@
     (pin "4")
     (instances
-      (project "FTDIBreakout"
+      (project "FT231x-Breakout"
         (path "/3ba8e31e-6a12-4b2c-b7ff-be557fb7bb2f"
           (reference "J2") (unit 1)
@@
     (pin "4")
     (instances
-      (project "FTDIBreakout"
+      (project "FT231x-Breakout"
         (path "/3ba8e31e-6a12-4b2c-b7ff-be557fb7bb2f"
           (reference "J1") (unit 1)
@@
     (pin "1")
     (instances
-      (project "FTDIBreakout"
+      (project "FT231x-Breakout"
         (path "/3ba8e31e-6a12-4b2c-b7ff-be557fb7bb2f"
           (reference "Q1") (unit 1)
@@
     (pin "1")
     (instances
-      (project "FTDIBreakout"
+      (project "FT231x-Breakout"
         (path "/3ba8e31e-6a12-4b2c-b7ff-be557fb7bb2f"
           (reference "#PWR07") (unit 1)
@@
     (pin "2")
     (instances
-      (project "FTDIBreakout"
+      (project "FT231x-Breakout"
         (path "/3ba8e31e-6a12-4b2c-b7ff-be557fb7bb2f"
           (reference "D1") (unit 1)
@@
     (pin "1")
     (instances
-      (project "FTDIBreakout"
+      (project "FT231x-Breakout"
         (path "/3ba8e31e-6a12-4b2c-b7ff-be557fb7bb2f"
           (reference "#PWR010") (unit 1)
@@
     (pin "1")
     (instances
-      (project "FTDIBreakout"
+      (project "FT231x-Breakout"
         (path "/3ba8e31e-6a12-4b2c-b7ff-be557fb7bb2f"
           (reference "#PWR011") (unit 1)
@@
     (pin "2")
     (instances
-      (project "FTDIBreakout"
+      (project "FT231x-Breakout"
         (path "/3ba8e31e-6a12-4b2c-b7ff-be557fb7bb2f"
           (reference "C4") (unit 1)
@@
     (pin "1")
     (instances
-      (project "FTDIBreakout"
+      (project "FT231x-Breakout"
         (path "/3ba8e31e-6a12-4b2c-b7ff-be557fb7bb2f"
           (reference "SW1") (unit 1)
@@
     (pin "1")
     (instances
-      (project "FTDIBreakout"
+      (project "FT231x-Breakout"
         (path "/3ba8e31e-6a12-4b2c-b7ff-be557fb7bb2f"
           (reference "R3") (unit 1)
@@
     (pin "1")
     (instances
-      (project "FTDIBreakout"
+      (project "FT231x-Breakout"
         (path "/3ba8e31e-6a12-4b2c-b7ff-be557fb7bb2f"
           (reference "#PWR01") (unit 1)
@@
     (pin "2")
     (instances
-      (project "FTDIBreakout"
+      (project "FT231x-Breakout"
         (path "/3ba8e31e-6a12-4b2c-b7ff-be557fb7bb2f"
           (reference "C5") (unit 1)
@@
     (pin "1")
     (instances
-      (project "FTDIBreakout"
+      (project "FT231x-Breakout"
         (path "/3ba8e31e-6a12-4b2c-b7ff-be557fb7bb2f"
           (reference "#PWR019") (unit 1)
@@
     (pin "1")
     (instances
-      (project "FTDIBreakout"
+      (project "FT231x-Breakout"
         (path "/3ba8e31e-6a12-4b2c-b7ff-be557fb7bb2f"
           (reference "#PWR021") (unit 1)
@@
     (pin "1")
     (instances
-      (project "FTDIBreakout"
+      (project "FT231x-Breakout"
         (path "/3ba8e31e-6a12-4b2c-b7ff-be557fb7bb2f"
           (reference "#PWR06") (unit 1)
@@
     (pin "2")
     (instances
-      (project "FTDIBreakout"
+      (project "FT231x-Breakout"
         (path "/3ba8e31e-6a12-4b2c-b7ff-be557fb7bb2f"
           (reference "C6") (unit 1)
@@
     (pin "1")
     (instances
-      (project "FTDIBreakout"
+      (project "FT231x-Breakout"
         (path "/3ba8e31e-6a12-4b2c-b7ff-be557fb7bb2f"
           (reference "J5") (unit 1)
@@
     (pin "1")
     (instances
-      (project "FTDIBreakout"
+      (project "FT231x-Breakout"
         (path "/3ba8e31e-6a12-4b2c-b7ff-be557fb7bb2f"
           (reference "#PWR05") (unit 1)
@@
     (pin "1")
     (instances
-      (project "FTDIBreakout"
+      (project "FT231x-Breakout"
         (path "/3ba8e31e-6a12-4b2c-b7ff-be557fb7bb2f"
           (reference "#PWR012") (unit 1)
@@
     (pin "1")
     (instances
-      (project "FTDIBreakout"
+      (project "FT231x-Breakout"
         (path "/3ba8e31e-6a12-4b2c-b7ff-be557fb7bb2f"
           (reference "#PWR03") (unit 1)
@@
     (pin "1")
     (instances
-      (project "FTDIBreakout"
+      (project "FT231x-Breakout"
         (path "/3ba8e31e-6a12-4b2c-b7ff-be557fb7bb2f"
           (reference "#PWR017") (unit 1)
@@
     (pin "1")
     (instances
-      (project "FTDIBreakout"
+      (project "FT231x-Breakout"
         (path "/3ba8e31e-6a12-4b2c-b7ff-be557fb7bb2f"
           (reference "R8") (unit 1)
@@
     (pin "1")
     (instances
-      (project "FTDIBreakout"
+      (project "FT231x-Breakout"
         (path "/3ba8e31e-6a12-4b2c-b7ff-be557fb7bb2f"
           (reference "J3") (unit 1)
@@
     (pin "2")
     (instances
-      (project "FTDIBreakout"
+      (project "FT231x-Breakout"
         (path "/3ba8e31e-6a12-4b2c-b7ff-be557fb7bb2f"
           (reference "C3") (unit 1)
@@
     (pin "1")
     (instances
-      (project "FTDIBreakout"
+      (project "FT231x-Breakout"
         (path "/3ba8e31e-6a12-4b2c-b7ff-be557fb7bb2f"
           (reference "R5") (unit 1)
@@
     (pin "1")
     (instances
-      (project "FTDIBreakout"
+      (project "FT231x-Breakout"
         (path "/3ba8e31e-6a12-4b2c-b7ff-be557fb7bb2f"
           (reference "Q2") (unit 1)
@@
     (pin "1")
     (instances
-      (project "FTDIBreakout"
+      (project "FT231x-Breakout"
         (path "/3ba8e31e-6a12-4b2c-b7ff-be557fb7bb2f"
           (reference "R4") (unit 1)
@@
     (pin "1")
     (instances
-      (project "FTDIBreakout"
+      (project "FT231x-Breakout"
         (path "/3ba8e31e-6a12-4b2c-b7ff-be557fb7bb2f"
           (reference "#PWR016") (unit 1)
